File: board/WiFiModem.kicad_pcb (KiCad board)
At the start: 2 copper layers, 88.9 x 61 mm, 46 parts, among them J1 DB9_Female, J2 DB25_Female, J3 Barrel_Jack_Switch, J4 PRG, SW1 SW_Push, SW2 SW_Push, U1 ESP-12E, U2 LM7805_TO220, U3 MAX232, U4 LT1117-3.3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

Commit message: Fix KiCAD 7.x DRC warnings.
Parts:
- U2: footprint Package_TO_SOT_THT:TO-220-3_Horizontal_TabDown -> Package_TO_SOT_THT:TO-220-3_Vertical
Connections:
- net +3V3 renamed +3.3V
Routing:
- net +3.3V: track 121.2 -> 119.9 mm
- net DCD: track 165.3 -> 164.0 mm
- net GPIO3: track 7.08 -> 5.88 mm
- net +5V: track 94.9 -> 94.1 mm
- net Net-(JP8-A): track 15.5 -> 14.8 mm
- net CTSB: track 53.7 -> 53.1 mm
- net Net-(U3-C1+): track 10.9 -> 10.4 mm
- net GPIO1: track 23.9 -> 23.3 mm
- net Net-(J4-Pin_2): track 5.74 -> 5.22 mm
- added copper zone on B.Cu, net GND
